Commit message: v6

File: otros/una_camara/turtlebot3_burger.gazebo.xacro (robot description, xacro)
@@ -3,5 +3,5 @@
   <xacro:arg name="laser_visual" default="true"/>
   <xacro:arg name="imu_visual"   default="false"/>
-  <xacro:arg name="camera_visual" default="false"/>
+  <xacro:arg name="camera_visual" default="true"/>
   <xacro:include filename="$(find realsense2_description)/urdf/_d435.urdf.xacro" />
   <xacro:include filename="$(find realsense2_description)/urdf/_d435.gazebo.xacro" />
@@ -132,6 +132,6 @@
       <visualize>$(arg camera_visual)</visualize>
       <camera>
-          <horizontal_fov>3.1</horizontal_fov>
-          <!-- <horizontal_fov>1.3439</horizontal_fov> -->
+          <horizontal_fov>3</horizontal_fov>
+          <!-- <horizontal_fov>1.34</horizontal_fov> -->
           <image>
               <width>1920</width>
@@ -171,47 +171,3 @@
     </sensor>
   </gazebo>
-<gazebo reference="back_camera_rgb_frame">
-    <sensor type="depth" name="realsense_R200">
-      <always_on>true</always_on>
-      <visualize>$(arg camera_visual)</visualize>
-      <camera name="back_camera">
-          <horizontal_fov>3.1</horizontal_fov>
-          <!-- <horizontal_fov>1.3439</horizontal_fov> -->
-          <image>
-              <width>1920</width>
-              <height>1080</height>
-              <format>R8G8B8</format>
-          </image>
-          <depth_camera></depth_camera>
-          <clip>
-              <near>0.03</near>
-              <far>100</far>
-          </clip>
-      </camera>
-      <plugin name="back_camera_controller" filename="libgazebo_ros_openni_kinect.so">
-        <baseline>0.2</baseline>
-        <alwaysOn>true</alwaysOn>
-        <updateRate>0.0</updateRate>
-        <cameraName>back_camera</cameraName>
-        <frameName>back_camera_rgb_optical_frame</frameName>
-        <imageTopicName>rgb/image_raw</imageTopicName>
-        <depthImageTopicName>depth/image_raw</depthImageTopicName>
-        <pointCloudTopicName>depth/points</pointCloudTopicName>
-        <cameraInfoTopicName>rgb/camera_info</cameraInfoTopicName>
-        <depthImageCameraInfoTopicName>depth/camera_info</depthImageCameraInfoTopicName>
-        <pointCloudCutoff>0.0</pointCloudCutoff>
-            <hackBaseline>0.07</hackBaseline>
-            <distortionK1>0.0</distortionK1>
-            <distortionK2>0.0</distortionK2>
-            <distortionK3>0.0</distortionK3>
-            <distortionT1>0.0</distortionT1>
-            <distortionT2>0.0</distortionT2>
-        <CxPrime>0.0</CxPrime>
-        <Cx>0.0</Cx>
-        <Cy>0.0</Cy>
-        <focalLength>0</focalLength>
-        <hackBaseline>0</hackBaseline>
-      </plugin>
-    </sensor>
-  </gazebo>
 </robot>

File: otros/una_camara/turtlebot3_burger.urdf.xacro (robot description, xacro)
@@ -147,5 +147,5 @@
   </link>
 <joint name="camera_joint" type="fixed">
-    <origin xyz="-0.032 0 0.172" rpy="0 0 0"/>
+    <origin xyz="-0.032 0 0.172" rpy="0 0 0.15"/>
     <parent link="base_link"/>
     <child link="camera_link"/>
@@ -200,50 +200,3 @@
   </joint>
   <link name="camera_depth_optical_frame"/>
-<!-- second camera -->
-<joint name="back_camera_joint" type="fixed">
-    <origin xyz="-0.082 0 0.172" rpy="0 0 3.1415"/>
-    <parent link="base_link"/>
-    <child link="back_camera_link"/>
-  </joint>
-  <link name="back_camera_link">
-    <visual>
-     <origin xyz="0 0 0" rpy="1.57 0 1.57"/>
-      <geometry>
-       <mesh filename="package://realsense2_description/meshes/d435.dae" />
-      </geometry>
-        <material name="gazebo_d435_aluminum">
-    	<color rgba="0.5 0.5 0.5 1"/>
-    	</material>
-    </visual>
-    <collision>
-      <origin xyz="0.015 0 -0.0065" rpy="0 0 0"/>
-      <geometry>
-        <box size="0.003 0.25 0.016"/>
-      </geometry>
-    </collision>
-  </link>
-  <joint name="back_camera_rgb_joint" type="fixed">
-    <origin xyz="${r200_cam_rgb_px} ${r200_cam_rgb_py} ${r200_cam_rgb_pz}" rpy="0 0 0"/>
-    <parent link="back_camera_link"/>
-    <child link="back_camera_rgb_frame"/>
-  </joint>
-  <link name="back_camera_rgb_frame"/>
-  <joint name="back_camera_rgb_optical_joint" type="fixed">
-    <origin xyz="0 0 0" rpy="-1.57 0 -1.57"/>
-    <parent link="back_camera_rgb_frame"/>
-    <child link="back_camera_rgb_optical_frame"/>
-  </joint>
-  <link name="back_camera_rgb_optical_frame"/>
-  <joint name="back_camera_depth_joint" type="fixed">
-    <origin xyz="0 0 0" rpy="0 0 0"/>
-    <parent link="back_camera_link"/>
-    <child link="back_camera_depth_frame"/>
-  </joint>
-  <link name="back_camera_depth_frame"/>
-  <joint name="back_camera_depth_optical_joint" type="fixed">
-    <origin xyz="0 0 0" rpy="-1.57 0 -1.57"/>
-    <parent link="back_camera_depth_frame"/>
-    <child link="back_camera_depth_optical_frame"/>
-  </joint>
-  <link name="back_camera_depth_optical_frame"/>
 </robot>
