Commit message: v5

File: src/turtlebot3/turtlebot3_description/urdf/turtlebot3_burger.urdf.xacro (robot description, xacro)
@@ -147,5 +147,5 @@
   </link>
 <joint name="camera_joint" type="fixed">
-    <origin xyz="-0.032 0 0.172" rpy="0 0 0"/>
+    <origin xyz="-0.032 0 0.172" rpy="0 0 0.15"/>
     <parent link="base_link"/>
     <child link="camera_link"/>

Commit message: v7

File: src/turtlebot3/turtlebot3_description/urdf/turtlebot3_burger.urdf.xacro (robot description, xacro)
@@ -162,5 +162,5 @@
     </visual>
     <collision>
-      <origin xyz="0.015 0 -0.0065" rpy="0 0 0"/>
+      <origin xyz="0.012 0 -0.0065" rpy="0 0 0"/>
       <geometry>
         <box size="0.003 0.25 0.016"/>
