Commit message: v4

File: src/turtlebot3/turtlebot3_description/urdf/turtlebot3_burger.gazebo.xacro (robot description, xacro)
@@ -133,4 +133,5 @@
       <camera>
           <horizontal_fov>3</horizontal_fov>
+          <!-- <horizontal_fov>1.34</horizontal_fov> -->
           <image>
               <width>1920</width>

File: src/turtlebot3/turtlebot3_description/urdf/turtlebot3_burger.urdf.xacro (robot description, xacro)
@@ -147,5 +147,5 @@
   </link>
 <joint name="camera_joint" type="fixed">
-    <origin xyz="0.064 0.0 0.19" rpy="0 0 0"/>
+    <origin xyz="-0.032 0 0.172" rpy="0 0 0"/>
     <parent link="base_link"/>
     <child link="camera_link"/>
@@ -162,5 +162,5 @@
     </visual>
     <collision>
-      <origin xyz="0.003 0.035 0.007" rpy="0 0 0"/>
+      <origin xyz="0.015 0 -0.0065" rpy="0 0 0"/>
       <geometry>
         <box size="0.003 0.25 0.016"/>

Commit message: v8

File: src/turtlebot3/turtlebot3_description/urdf/turtlebot3_burger.gazebo.xacro (robot description, xacro)
@@ -133,4 +133,5 @@
       <camera>
           <horizontal_fov>3.1</horizontal_fov>
+          <!-- <horizontal_fov>3.1 </horizontal_fov> -->
           <!-- <horizontal_fov>1.3439</horizontal_fov> -->
           <image>
@@ -156,5 +157,5 @@
         <cameraInfoTopicName>rgb/camera_info</cameraInfoTopicName>
         <depthImageCameraInfoTopicName>depth/camera_info</depthImageCameraInfoTopicName>
-        <pointCloudCutoff>0.0</pointCloudCutoff>
+        <pointCloudCutoff>-0.01</pointCloudCutoff>
             <hackBaseline>0.07</hackBaseline>
             <distortionK1>0.0</distortionK1>
@@ -200,5 +201,5 @@
         <cameraInfoTopicName>rgb/camera_info</cameraInfoTopicName>
         <depthImageCameraInfoTopicName>depth/camera_info</depthImageCameraInfoTopicName>
-        <pointCloudCutoff>0.0</pointCloudCutoff>
+        <pointCloudCutoff>-0.01</pointCloudCutoff>
             <hackBaseline>0.07</hackBaseline>
             <distortionK1>0.0</distortionK1>

File: src/turtlebot3/turtlebot3_description/urdf/turtlebot3_burger.urdf.xacro (robot description, xacro)
@@ -162,5 +162,5 @@
     </visual>
     <collision>
-      <origin xyz="0.012 0 -0.0065" rpy="0 0 0"/>
+      <origin xyz="0.015 0 -0.0065" rpy="0 0 0"/>
       <geometry>
         <box size="0.003 0.25 0.016"/>
@@ -217,5 +217,5 @@
     </visual>
     <collision>
-      <origin xyz="0.015 0 -0.0065" rpy="0 0 0"/>
+      <origin xyz="-0.065 0 -0.0065" rpy="0 0 0"/>
       <geometry>
         <box size="0.003 0.25 0.016"/>

Commit message: v12

File: src/turtlebot3/turtlebot3_description/urdf/turtlebot3_burger.gazebo.xacro (robot description, xacro)
@@ -127,92 +127,3 @@
     </sensor>
   </gazebo>
-<gazebo reference="camera_rgb_frame">
-    <sensor type="depth" name="realsense_R200">
-      <always_on>true</always_on>
-      <visualize>$(arg camera_visual)</visualize>
-      <camera>
-          <horizontal_fov>3.1</horizontal_fov>
-          <!-- <horizontal_fov>3.1 </horizontal_fov> -->
-          <!-- <horizontal_fov>1.3439</horizontal_fov> -->
-          <image>
-              <width>1920</width>
-              <height>1080</height>
-              <format>R8G8B8</format>
-          </image>
-          <depth_camera></depth_camera>
-          <clip>
-              <near>0.03</near>
-              <far>100</far>
-          </clip>
-      </camera>
-      <plugin name="camera_controller" filename="libgazebo_ros_openni_kinect.so">
-        <baseline>0.2</baseline>
-        <alwaysOn>true</alwaysOn>
-        <updateRate>0.0</updateRate>
-        <cameraName>camera</cameraName>
-        <frameName>camera_rgb_optical_frame</frameName>
-        <imageTopicName>rgb/image_raw</imageTopicName>
-        <depthImageTopicName>depth/image_raw</depthImageTopicName>
-        <pointCloudTopicName>depth/points</pointCloudTopicName>
-        <cameraInfoTopicName>rgb/camera_info</cameraInfoTopicName>
-        <depthImageCameraInfoTopicName>depth/camera_info</depthImageCameraInfoTopicName>
-        <pointCloudCutoff>-0.01</pointCloudCutoff>
-            <hackBaseline>0.07</hackBaseline>
-            <distortionK1>0.0</distortionK1>
-            <distortionK2>0.0</distortionK2>
-            <distortionK3>0.0</distortionK3>
-            <distortionT1>0.0</distortionT1>
-            <distortionT2>0.0</distortionT2>
-        <CxPrime>0.0</CxPrime>
-        <Cx>0.0</Cx>
-        <Cy>0.0</Cy>
-        <focalLength>0</focalLength>
-        <hackBaseline>0</hackBaseline>
-      </plugin>
-    </sensor>
-  </gazebo>
-<gazebo reference="back_camera_rgb_frame">
-    <sensor type="depth" name="realsense_R200">
-      <always_on>true</always_on>
-      <visualize>$(arg camera_visual)</visualize>
-      <camera name="back_camera">
-          <horizontal_fov>3.1</horizontal_fov>
-          <!-- <horizontal_fov>1.3439</horizontal_fov> -->
-          <image>
-              <width>1920</width>
-              <height>1080</height>
-              <format>R8G8B8</format>
-          </image>
-          <depth_camera></depth_camera>
-          <clip>
-              <near>0.03</near>
-              <far>100</far>
-          </clip>
-      </camera>
-      <plugin name="back_camera_controller" filename="libgazebo_ros_openni_kinect.so">
-        <baseline>0.2</baseline>
-        <alwaysOn>true</alwaysOn>
-        <updateRate>0.0</updateRate>
-        <cameraName>back_camera</cameraName>
-        <frameName>back_camera_rgb_optical_frame</frameName>
-        <imageTopicName>rgb/image_raw</imageTopicName>
-        <depthImageTopicName>depth/image_raw</depthImageTopicName>
-        <pointCloudTopicName>depth/points</pointCloudTopicName>
-        <cameraInfoTopicName>rgb/camera_info</cameraInfoTopicName>
-        <depthImageCameraInfoTopicName>depth/camera_info</depthImageCameraInfoTopicName>
-        <pointCloudCutoff>-0.01</pointCloudCutoff>
-            <hackBaseline>0.07</hackBaseline>
-            <distortionK1>0.0</distortionK1>
-            <distortionK2>0.0</distortionK2>
-            <distortionK3>0.0</distortionK3>
-            <distortionT1>0.0</distortionT1>
-            <distortionT2>0.0</distortionT2>
-        <CxPrime>0.0</CxPrime>
-        <Cx>0.0</Cx>
-        <Cy>0.0</Cy>
-        <focalLength>0</focalLength>
-        <hackBaseline>0</hackBaseline>
-      </plugin>
-    </sensor>
-  </gazebo>
 </robot>

File: src/turtlebot3/turtlebot3_description/urdf/turtlebot3_burger.urdf.xacro (robot description, xacro)
@@ -146,104 +146,3 @@
     </inertial>
   </link>
-<joint name="camera_joint" type="fixed">
-    <origin xyz="-0.032 0 0.172" rpy="0 0 0"/>
-    <parent link="base_link"/>
-    <child link="camera_link"/>
-  </joint>
-  <link name="camera_link">
-    <visual>
-     <origin xyz="0 0 0" rpy="1.57 0 1.57"/>
-      <geometry>
-       <mesh filename="package://realsense2_description/meshes/d435.dae" />
-      </geometry>
-        <material name="gazebo_d435_aluminum">
-    	<color rgba="0.5 0.5 0.5 1"/>
-    	</material>
-    </visual>
-    <collision>
-      <origin xyz="0.015 0 -0.0065" rpy="0 0 0"/>
-      <geometry>
-        <box size="0.003 0.25 0.016"/>
-      </geometry>
-    </collision>
-    <!-- This inertial field needs doesn't contain reliable data!! -->
-<!--   <inertial>
-      <mass value="0.564" />
-      <origin xyz="0 0 0" />
-      <inertia ixx="0.003881243" ixy="0.0" ixz="0.0"
-               iyy="0.000498940" iyz="0.0"
-               izz="0.003879257" />
-    </inertial>-->
-  </link>
-  <joint name="camera_rgb_joint" type="fixed">
-    <origin xyz="${r200_cam_rgb_px} ${r200_cam_rgb_py} ${r200_cam_rgb_pz}" rpy="0 0 0"/>
-    <parent link="camera_link"/>
-    <child link="camera_rgb_frame"/>
-  </joint>
-  <link name="camera_rgb_frame"/>
-  <joint name="camera_rgb_optical_joint" type="fixed">
-    <origin xyz="0 0 0" rpy="-1.57 0 -1.57"/>
-    <parent link="camera_rgb_frame"/>
-    <child link="camera_rgb_optical_frame"/>
-  </joint>
-  <link name="camera_rgb_optical_frame"/>
-  <joint name="camera_depth_joint" type="fixed">
-    <origin xyz="0 0 0" rpy="0 0 0"/>
-    <parent link="camera_link"/>
-    <child link="camera_depth_frame"/>
-  </joint>
-  <link name="camera_depth_frame"/>
-  <joint name="camera_depth_optical_joint" type="fixed">
-    <origin xyz="0 0 0" rpy="-1.57 0 -1.57"/>
-    <parent link="camera_depth_frame"/>
-    <child link="camera_depth_optical_frame"/>
-  </joint>
-  <link name="camera_depth_optical_frame"/>
-<!-- second camera -->
-<joint name="back_camera_joint" type="fixed">
-    <origin xyz="-0.082 0 0.172" rpy="0 0 3.1415"/>
-    <parent link="base_link"/>
-    <child link="back_camera_link"/>
-  </joint>
-  <link name="back_camera_link">
-    <visual>
-     <origin xyz="0 0 0" rpy="1.57 0 1.57"/>
-      <geometry>
-       <mesh filename="package://realsense2_description/meshes/d435.dae" />
-      </geometry>
-        <material name="gazebo_d435_aluminum">
-    	<color rgba="0.5 0.5 0.5 1"/>
-    	</material>
-    </visual>
-    <collision>
-      <origin xyz="-0.065 0 -0.0065" rpy="0 0 0"/>
-      <geometry>
-        <box size="0.003 0.25 0.016"/>
-      </geometry>
-    </collision>
-  </link>
-  <joint name="back_camera_rgb_joint" type="fixed">
-    <origin xyz="${r200_cam_rgb_px} ${r200_cam_rgb_py} ${r200_cam_rgb_pz}" rpy="0 0 0"/>
-    <parent link="back_camera_link"/>
-    <child link="back_camera_rgb_frame"/>
-  </joint>
-  <link name="back_camera_rgb_frame"/>
-  <joint name="back_camera_rgb_optical_joint" type="fixed">
-    <origin xyz="0 0 0" rpy="-1.57 0 -1.57"/>
-    <parent link="back_camera_rgb_frame"/>
-    <child link="back_camera_rgb_optical_frame"/>
-  </joint>
-  <link name="back_camera_rgb_optical_frame"/>
-  <joint name="back_camera_depth_joint" type="fixed">
-    <origin xyz="0 0 0" rpy="0 0 0"/>
-    <parent link="back_camera_link"/>
-    <child link="back_camera_depth_frame"/>
-  </joint>
-  <link name="back_camera_depth_frame"/>
-  <joint name="back_camera_depth_optical_joint" type="fixed">
-    <origin xyz="0 0 0" rpy="-1.57 0 -1.57"/>
-    <parent link="back_camera_depth_frame"/>
-    <child link="back_camera_depth_optical_frame"/>
-  </joint>
-  <link name="back_camera_depth_optical_frame"/>
 </robot>

File: src/turtlebot3/turtlebot3_description/urdf/turtlebot3_burger_1cam180.gazebo.xacro (robot description, xacro)
@@ -95,5 +95,5 @@
     </plugin>
   </gazebo>
-  <gazebo reference="base_scan">
+  <!-- <gazebo reference="base_scan">
     <material>Gazebo/FlatBlack</material>
     <sensor type="ray" name="lds_lfcd_sensor">
@@ -126,5 +126,5 @@
       </plugin>
     </sensor>
-  </gazebo>
+  </gazebo> -->
 <gazebo reference="camera_rgb_frame">
     <sensor type="depth" name="realsense_R200">
@@ -135,6 +135,6 @@
           <!-- <horizontal_fov>1.3439</horizontal_fov> -->
           <image>
-              <width>1920</width>
-              <height>1080</height>
+              <width>640</width>
+              <height>480</height>
               <format>R8G8B8</format>
           </image>

File: src/turtlebot3/turtlebot3_description/urdf/turtlebot3_burger_1cam180.urdf.xacro (robot description, xacro)
@@ -119,5 +119,5 @@
   </joint>
   <link name="imu_link"/>
-  <joint name="scan_joint" type="fixed">
+  <!-- <joint name="scan_joint" type="fixed">
     <parent link="base_link"/>
     <child link="base_scan"/>
@@ -145,5 +145,5 @@
                izz="0.001" />
     </inertial>
-  </link>
+  </link> -->
 <joint name="camera_joint" type="fixed">
     <origin xyz="-0.032 0 0.172" rpy="0 0 0.0"/>

File: src/turtlebot3/turtlebot3_description/urdf/turtlebot3_burger_1cam77.gazebo.xacro (robot description, xacro)
@@ -95,5 +95,5 @@
     </plugin>
   </gazebo>
-  <gazebo reference="base_scan">
+  <!-- <gazebo reference="base_scan">
     <material>Gazebo/FlatBlack</material>
     <sensor type="ray" name="lds_lfcd_sensor">
@@ -126,5 +126,5 @@
       </plugin>
     </sensor>
-  </gazebo>
+  </gazebo> -->
 <gazebo reference="camera_rgb_frame">
     <sensor type="depth" name="realsense_R200">
@@ -132,9 +132,9 @@
       <visualize>$(arg camera_visual)</visualize>
       <camera>
-          <horizontal_fov>1.34390352404</horizontal_fov>
+          <horizontal_fov>1.570796</horizontal_fov>
           <!-- <horizontal_fov>1.3439</horizontal_fov> -->
           <image>
-              <width>1920</width>
-              <height>1080</height>
+              <width>640</width>
+              <height>480</height>
               <format>R8G8B8</format>
           </image>

File: src/turtlebot3/turtlebot3_description/urdf/turtlebot3_burger_1cam77.urdf.xacro (robot description, xacro)
@@ -119,5 +119,5 @@
   </joint>
   <link name="imu_link"/>
-  <joint name="scan_joint" type="fixed">
+  <!-- <joint name="scan_joint" type="fixed">
     <parent link="base_link"/>
     <child link="base_scan"/>
@@ -145,5 +145,5 @@
                izz="0.001" />
     </inertial>
-  </link>
+  </link> -->
 <joint name="camera_joint" type="fixed">
     <origin xyz="-0.032 0 0.172" rpy="0 0 0.0"/>

File: src/turtlebot3/turtlebot3_description/urdf/turtlebot3_burger_2cam.gazebo.xacro (robot description, xacro)
@@ -135,6 +135,6 @@
           <!-- <horizontal_fov>1.3439</horizontal_fov> -->
           <image>
-              <width>1280</width>
-              <height>720</height>
+              <width>640</width>
+              <height>480</height>
               <format>R8G8B8</format>
           </image>
@@ -178,6 +178,6 @@
           <horizontal_fov>3.1</horizontal_fov>
           <image>
-              <width>1280</width>
-              <height>720</height>
+              <width>640</width>
+              <height>480</height>
               <format>R8G8B8</format>
           </image>
