Commit message: v13

File: src/turtlebot3/turtlebot3_description/urdf/turtlebot3_burger_1cam120.gazebo.xacro (robot description, xacro)
@@ -95,10 +95,10 @@
     </plugin>
   </gazebo>
-  <!-- <gazebo reference="base_scan">
+  <gazebo reference="base_scan">
     <material>Gazebo/FlatBlack</material>
     <sensor type="ray" name="lds_lfcd_sensor">
       <pose>0 0 0 0 0 0</pose>
       <visualize>$(arg laser_visual)</visualize>
-      <update_rate>5</update_rate>
+      <update_rate>6.8</update_rate>
       <ray>
         <scan>
@@ -126,5 +126,5 @@
       </plugin>
     </sensor>
-  </gazebo> -->
+  </gazebo>
 <gazebo reference="camera_rgb_frame">
     <sensor type="depth" name="realsense_R200">

File: src/turtlebot3/turtlebot3_description/urdf/turtlebot3_burger_1cam120.urdf.xacro (robot description, xacro)
@@ -119,5 +119,5 @@
   </joint>
   <link name="imu_link"/>
-  <!-- <joint name="scan_joint" type="fixed">
+  <joint name="scan_joint" type="fixed">
     <parent link="base_link"/>
     <child link="base_scan"/>
@@ -145,5 +145,5 @@
                izz="0.001" />
     </inertial>
-  </link> -->
+  </link>
 <joint name="camera_joint" type="fixed">
     <origin xyz="-0.032 0 0.172" rpy="0 0 0"/>

File: src/turtlebot3/turtlebot3_description/urdf/turtlebot3_burger_1cam150.gazebo.xacro (robot description, xacro)
@@ -95,10 +95,10 @@
     </plugin>
   </gazebo>
-  <!-- <gazebo reference="base_scan">
+  <gazebo reference="base_scan">
     <material>Gazebo/FlatBlack</material>
     <sensor type="ray" name="lds_lfcd_sensor">
       <pose>0 0 0 0 0 0</pose>
       <visualize>$(arg laser_visual)</visualize>
-      <update_rate>5</update_rate>
+      <update_rate>6.8</update_rate>
       <ray>
         <scan>
@@ -126,5 +126,5 @@
       </plugin>
     </sensor>
-  </gazebo> -->
+  </gazebo>
 <gazebo reference="camera_rgb_frame">
     <sensor type="depth" name="realsense_R200">

File: src/turtlebot3/turtlebot3_description/urdf/turtlebot3_burger_1cam150.urdf.xacro (robot description, xacro)
@@ -119,5 +119,5 @@
   </joint>
   <link name="imu_link"/>
-  <!-- <joint name="scan_joint" type="fixed">
+  <joint name="scan_joint" type="fixed">
     <parent link="base_link"/>
     <child link="base_scan"/>
@@ -145,5 +145,5 @@
                izz="0.001" />
     </inertial>
-  </link> -->
+  </link>
 <joint name="camera_joint" type="fixed">
     <origin xyz="-0.032 0 0.172" rpy="0 0 0"/>

File: src/turtlebot3/turtlebot3_description/urdf/turtlebot3_burger_1cam180.gazebo.xacro (robot description, xacro)
@@ -95,10 +95,10 @@
     </plugin>
   </gazebo>
-  <!-- <gazebo reference="base_scan">
+  <gazebo reference="base_scan">
     <material>Gazebo/FlatBlack</material>
     <sensor type="ray" name="lds_lfcd_sensor">
       <pose>0 0 0 0 0 0</pose>
       <visualize>$(arg laser_visual)</visualize>
-      <update_rate>5</update_rate>
+      <update_rate>6.8</update_rate>
       <ray>
         <scan>
@@ -126,5 +126,5 @@
       </plugin>
     </sensor>
-  </gazebo> -->
+  </gazebo>
 <gazebo reference="camera_rgb_frame">
     <sensor type="depth" name="realsense_R200">

File: src/turtlebot3/turtlebot3_description/urdf/turtlebot3_burger_1cam180.urdf.xacro (robot description, xacro)
@@ -119,5 +119,5 @@
   </joint>
   <link name="imu_link"/>
-  <!-- <joint name="scan_joint" type="fixed">
+  <joint name="scan_joint" type="fixed">
     <parent link="base_link"/>
     <child link="base_scan"/>
@@ -145,5 +145,5 @@
                izz="0.001" />
     </inertial>
-  </link> -->
+  </link>
 <joint name="camera_joint" type="fixed">
     <origin xyz="-0.032 0 0.172" rpy="0 0 0.0"/>

File: src/turtlebot3/turtlebot3_description/urdf/turtlebot3_burger_1cam77.gazebo.xacro (robot description, xacro)
@@ -95,10 +95,10 @@
     </plugin>
   </gazebo>
-  <!-- <gazebo reference="base_scan">
+  <gazebo reference="base_scan">
     <material>Gazebo/FlatBlack</material>
     <sensor type="ray" name="lds_lfcd_sensor">
       <pose>0 0 0 0 0 0</pose>
       <visualize>$(arg laser_visual)</visualize>
-      <update_rate>5</update_rate>
+      <update_rate>6.8</update_rate>
       <ray>
         <scan>
@@ -126,5 +126,5 @@
       </plugin>
     </sensor>
-  </gazebo> -->
+  </gazebo>
 <gazebo reference="camera_rgb_frame">
     <sensor type="depth" name="realsense_R200">

File: src/turtlebot3/turtlebot3_description/urdf/turtlebot3_burger_1cam77.urdf.xacro (robot description, xacro)
@@ -119,5 +119,5 @@
   </joint>
   <link name="imu_link"/>
-  <!-- <joint name="scan_joint" type="fixed">
+  <joint name="scan_joint" type="fixed">
     <parent link="base_link"/>
     <child link="base_scan"/>
@@ -145,5 +145,5 @@
                izz="0.001" />
     </inertial>
-  </link> -->
+  </link>
 <joint name="camera_joint" type="fixed">
     <origin xyz="-0.032 0 0.172" rpy="0 0 0.0"/>

File: src/turtlebot3/turtlebot3_description/urdf/turtlebot3_burger_1cam90.gazebo.xacro (robot description, xacro)
@@ -95,10 +95,10 @@
     </plugin>
   </gazebo>
-  <!-- <gazebo reference="base_scan">
+  <gazebo reference="base_scan">
     <material>Gazebo/FlatBlack</material>
     <sensor type="ray" name="lds_lfcd_sensor">
       <pose>0 0 0 0 0 0</pose>
       <visualize>$(arg laser_visual)</visualize>
-      <update_rate>5</update_rate>
+      <update_rate>6.8</update_rate>
       <ray>
         <scan>
@@ -126,5 +126,5 @@
       </plugin>
     </sensor>
-  </gazebo> -->
+  </gazebo>
 <gazebo reference="camera_rgb_frame">
     <sensor type="depth" name="realsense_R200">

File: src/turtlebot3/turtlebot3_description/urdf/turtlebot3_burger_1cam90.urdf.xacro (robot description, xacro)
@@ -119,5 +119,5 @@
   </joint>
   <link name="imu_link"/>
-  <!-- <joint name="scan_joint" type="fixed">
+  <joint name="scan_joint" type="fixed">
     <parent link="base_link"/>
     <child link="base_scan"/>
@@ -145,5 +145,5 @@
                izz="0.001" />
     </inertial>
-  </link> -->
+  </link>
 <joint name="camera_joint" type="fixed">
     <origin xyz="-0.032 0 0.172" rpy="0 0 0"/>
