Commit message: v11

File: src/send/realsense2_description/urdf/_d435.gazebo.xacro (robot description, xacro)
@@ -133,5 +133,5 @@
         <pointCloud>${publish_pointcloud}</pointCloud>
         <pointCloudTopicName>depth/color/points</pointCloudTopicName>
-        <pointCloudCutoff>0.25</pointCloudCutoff>
+        <pointCloudCutoff>0.0</pointCloudCutoff>
         <pointCloudCutoffMax>9.0</pointCloudCutoffMax>
       </plugin>

File: src/turtlebot3/turtlebot3_description/urdf/turtlebot3_burger_2cam.gazebo.xacro (robot description, xacro)
@@ -95,5 +95,5 @@
     </plugin>
   </gazebo>
-  <gazebo reference="base_scan">
+  <!-- <gazebo reference="base_scan">
     <material>Gazebo/FlatBlack</material>
     <sensor type="ray" name="lds_lfcd_sensor">
@@ -126,5 +126,5 @@
       </plugin>
     </sensor>
-  </gazebo>
+  </gazebo> -->
   <gazebo reference="camera_rgb_frame">
     <sensor type="depth" name="realsense_R200">
@@ -135,6 +135,6 @@
           <!-- <horizontal_fov>1.3439</horizontal_fov> -->
           <image>
-              <width>1920</width>
-              <height>1080</height>
+              <width>1280</width>
+              <height>720</height>
               <format>R8G8B8</format>
           </image>
@@ -178,6 +178,6 @@
           <horizontal_fov>3.1</horizontal_fov>
           <image>
-              <width>1920</width>
-              <height>1080</height>
+              <width>1280</width>
+              <height>720</height>
               <format>R8G8B8</format>
           </image>

File: src/turtlebot3/turtlebot3_description/urdf/turtlebot3_burger_2cam.urdf.xacro (robot description, xacro)
@@ -119,5 +119,5 @@
   </joint>
   <link name="imu_link"/>
-  <joint name="scan_joint" type="fixed">
+  <!-- <joint name="scan_joint" type="fixed">
     <parent link="base_link"/>
     <child link="base_scan"/>
@@ -145,5 +145,5 @@
                izz="0.001" />
     </inertial>
-  </link>
+  </link> -->
   <joint name="camera_joint" type="fixed">
     <origin xyz="-0.032 0 0.2" rpy="0 0 0"/>
